Commit message: Update omni_roller.xacro

File: 3_Wheel/urdf/omni_roller.xacro (robot description, xacro)
@@ -9,10 +9,10 @@
     <visual>
       <geometry>
-        <cylinder radius="0.01" length="0.03"/>
+        <cylinder radius="0.012" length="0.0185"/>
       </geometry>
     </visual>
     <collision>
       <geometry>
-        <cylinder radius="0.01" length="0.03"/>
+        <cylinder radius="0.012" length="0.0185"/>
       </geometry>
     </collision>
