Commit message: update

File: 4_Wheel/quadwheel/model/main.xacro (robot description, xacro)
@@ -31,3 +31,44 @@
   <xacro:connector name="3" parent="chassis" xyz="-0.228 -0.228 0.01" rpy="1.57 0 -3.9270" GAZEBO_color = "Gazebo/Green"/>
   <xacro:connector name="4" parent="chassis" xyz="-0.228 0.228 0.01" rpy="1.57 0 -5.4978" GAZEBO_color = "Gazebo/Yellow"/>
+  <!-- Motors -->
+  <transmission name="tran1">
+    <type>transmission_interface/SimpleTransmission</type>
+    <joint name="chassis_C1_joint">
+      <hardwareInterface>hardware_interface/EffortJointInterface</hardwareInterface>
+    </joint>
+    <actuator name="motor1">
+      <hardwareInterface>hardware_interface/EffortJointInterface</hardwareInterface>
+      <mechanicalReduction>1</mechanicalReduction>
+    </actuator>
+  </transmission>
+  <transmission name="tran2">
+    <type>transmission_interface/SimpleTransmission</type>
+    <joint name="chassis_C2_joint">
+      <hardwareInterface>hardware_interface/EffortJointInterface</hardwareInterface>
+    </joint>
+    <actuator name="motor2">
+      <hardwareInterface>hardware_interface/EffortJointInterface</hardwareInterface>
+      <mechanicalReduction>1</mechanicalReduction>
+    </actuator>
+  </transmission>
+  <transmission name="tran3">
+    <type>transmission_interface/SimpleTransmission</type>
+    <joint name="chassis_C3_joint">
+      <hardwareInterface>hardware_interface/EffortJointInterface</hardwareInterface>
+    </joint>
+    <actuator name="motor3">
+      <hardwareInterface>hardware_interface/EffortJointInterface</hardwareInterface>
+      <mechanicalReduction>1</mechanicalReduction>
+    </actuator>
+  </transmission>
+  <transmission name="tran4">
+    <type>transmission_interface/SimpleTransmission</type>
+    <joint name="chassis_C4_joint">
+      <hardwareInterface>hardware_interface/EffortJointInterface</hardwareInterface>
+    </joint>
+    <actuator name="motor4">
+      <hardwareInterface>hardware_interface/EffortJointInterface</hardwareInterface>
+      <mechanicalReduction>1</mechanicalReduction>
+    </actuator>
+  </transmission>
 </robot>

File: 4_Wheel/quadwheel/model/rim.xacro (robot description, xacro)
@@ -22,22 +22,22 @@
     <origin xyz = "${xyz}" rpy = "${rpy}"/>
   </joint>
-<xacro:roller name="1" parent="${name}"  xyz="0.0415 0 -0.0102" rpy="1.57 0 0" GAZEBO_color = "${GAZEBO_color}"/>
-<xacro:roller name="2" parent="${name}"  xyz="0.0390 0.0142 0.0102" rpy="1.57 0 0.3491" GAZEBO_color = "${GAZEBO_color}"/>
-<xacro:roller name="3" parent="${name}"  xyz="0.0318 0.0267 -0.0102" rpy="1.57 0 0.6981" GAZEBO_color = "${GAZEBO_color}"/>
-<xacro:roller name="4" parent="${name}"  xyz="0.0208 0.0359 0.0102" rpy="1.57 0 1.0472" GAZEBO_color = "${GAZEBO_color}"/>
-<xacro:roller name="5" parent="${name}"  xyz="0.0072 0.0409 -0.0102" rpy="1.57 0 1.3963" GAZEBO_color = "${GAZEBO_color}"/>
-<xacro:roller name="6" parent="${name}"  xyz="-0.0072 0.0409 0.0102" rpy="1.57 0 1.7453" GAZEBO_color = "${GAZEBO_color}"/>
-<xacro:roller name="7" parent="${name}"  xyz="-0.0208 0.0359 -0.0102" rpy="1.57 0 2.0944" GAZEBO_color = "${GAZEBO_color}"/>
-<xacro:roller name="8" parent="${name}"  xyz="-0.0318 0.0267 0.0102" rpy="1.57 0 2.4435" GAZEBO_color = "${GAZEBO_color}"/>
-<xacro:roller name="9" parent="${name}"  xyz="-0.0390 0.0142 -0.0102" rpy="1.57 0 2.7925" GAZEBO_color = "${GAZEBO_color}"/>
-<xacro:roller name="10" parent="${name}"  xyz="-0.0415 0 0.0102" rpy="1.57 0 3.1416" GAZEBO_color = "${GAZEBO_color}"/>
-<xacro:roller name="11" parent="${name}"  xyz="-0.0390 -0.0142 -0.0102" rpy="1.57 0 3.4907" GAZEBO_color = "${GAZEBO_color}"/>
-<xacro:roller name="12" parent="${name}"  xyz="-0.0318 -0.0267 0.0102" rpy="1.57 0 3.8397" GAZEBO_color = "${GAZEBO_color}"/>
-<xacro:roller name="13" parent="${name}"  xyz="-0.0208 -0.0359 -0.0102" rpy="1.57 0 4.1888" GAZEBO_color = "${GAZEBO_color}"/>
-<xacro:roller name="14" parent="${name}"  xyz="-0.00072 -0.0409 0.0102" rpy="1.57 0 4.5379" GAZEBO_color = "${GAZEBO_color}"/>
-<xacro:roller name="15" parent="${name}"  xyz="0.0072 -0.0409 -0.0102" rpy="1.57 0 4.8869" GAZEBO_color = "${GAZEBO_color}"/>
-<xacro:roller name="16" parent="${name}"  xyz="0.0208 -0.0359 0.0102" rpy="1.57 0 5.2360" GAZEBO_color = "${GAZEBO_color}"/>
-<xacro:roller name="17" parent="${name}"  xyz="0.0318 -0.0267 -0.0102" rpy="1.57 0 5.5851" GAZEBO_color = "${GAZEBO_color}"/>
-<xacro:roller name="18" parent="${name}"  xyz="0.0390 -0.0142 0.0102" rpy="1.57 0 5.9341" GAZEBO_color = "${GAZEBO_color}"/>
+<xacro:roller name="1" parent="${name}"  xyz="0.0415 0 -0.0284" rpy="1.57 0 0" GAZEBO_color = "${GAZEBO_color}"/>
+<xacro:roller name="2" parent="${name}"  xyz="0.0390 0.0142 -0.008" rpy="1.57 0 0.3491" GAZEBO_color = "${GAZEBO_color}"/>
+<xacro:roller name="3" parent="${name}"  xyz="0.0318 0.0267 -0.0284" rpy="1.57 0 0.6981" GAZEBO_color = "${GAZEBO_color}"/>
+<xacro:roller name="4" parent="${name}"  xyz="0.0208 0.0359 -0.008" rpy="1.57 0 1.0472" GAZEBO_color = "${GAZEBO_color}"/>
+<xacro:roller name="5" parent="${name}"  xyz="0.0072 0.0409 -0.0284" rpy="1.57 0 1.3963" GAZEBO_color = "${GAZEBO_color}"/>
+<xacro:roller name="6" parent="${name}"  xyz="-0.0072 0.0409 -0.008" rpy="1.57 0 1.7453" GAZEBO_color = "${GAZEBO_color}"/>
+<xacro:roller name="7" parent="${name}"  xyz="-0.0208 0.0359 -0.0284" rpy="1.57 0 2.0944" GAZEBO_color = "${GAZEBO_color}"/>
+<xacro:roller name="8" parent="${name}"  xyz="-0.0318 0.0267 -0.008" rpy="1.57 0 2.4435" GAZEBO_color = "${GAZEBO_color}"/>
+<xacro:roller name="9" parent="${name}"  xyz="-0.0390 0.0142 -0.0284" rpy="1.57 0 2.7925" GAZEBO_color = "${GAZEBO_color}"/>
+<xacro:roller name="10" parent="${name}"  xyz="-0.0415 0 -0.008" rpy="1.57 0 3.1416" GAZEBO_color = "${GAZEBO_color}"/>
+<xacro:roller name="11" parent="${name}"  xyz="-0.0390 -0.0142 -0.0284" rpy="1.57 0 3.4907" GAZEBO_color = "${GAZEBO_color}"/>
+<xacro:roller name="12" parent="${name}"  xyz="-0.0318 -0.0267 -0.008" rpy="1.57 0 3.8397" GAZEBO_color = "${GAZEBO_color}"/>
+<xacro:roller name="13" parent="${name}"  xyz="-0.0208 -0.0359 -0.0284" rpy="1.57 0 4.1888" GAZEBO_color = "${GAZEBO_color}"/>
+<xacro:roller name="14" parent="${name}"  xyz="-0.00072 -0.0409 -0.008" rpy="1.57 0 4.5379" GAZEBO_color = "${GAZEBO_color}"/>
+<xacro:roller name="15" parent="${name}"  xyz="0.0072 -0.0409 -0.0284" rpy="1.57 0 4.8869" GAZEBO_color = "${GAZEBO_color}"/>
+<xacro:roller name="16" parent="${name}"  xyz="0.0208 -0.0359 -0.008" rpy="1.57 0 5.2360" GAZEBO_color = "${GAZEBO_color}"/>
+<xacro:roller name="17" parent="${name}"  xyz="0.0318 -0.0267 -0.0284" rpy="1.57 0 5.5851" GAZEBO_color = "${GAZEBO_color}"/>
+<xacro:roller name="18" parent="${name}"  xyz="0.0390 -0.0142 -0.008" rpy="1.57 0 5.9341" GAZEBO_color = "${GAZEBO_color}"/>
 <gazebo reference="rim_${name}_link">
   <mu>0.2</mu>

File: 4_Wheel/quadwheel/model/roller.xacro (robot description, xacro)
@@ -4,10 +4,10 @@
   <link name="roller_${name}_rim_${parent}_link">
     <inertial>
-      <origin xyz="0 -0.0182 0" rpy="0 0 0" />
+      <origin xyz="0 0 0" rpy="0 0 0" />
       <inertia ixx="1e-6" ixy="0.0" ixz="0.0" iyy="1e-6" iyz="0.0" izz="1e-7"/>
       <mass value="0.010"/>
     </inertial>
     <visual>
-      <origin xyz="0 -0.0182 0" rpy="0 0 0" />
+      <origin xyz="0 0 0" rpy="0 0 0" />
       <geometry>
         <cylinder radius="0.01" length="0.03"/>
@@ -15,5 +15,5 @@
     </visual>
     <collision>
-      <origin xyz="0 -0.0182 0" rpy="0 0 0" />
+      <origin xyz="0 0 0" rpy="0 0 0" />
       <geometry>
         <cylinder radius="0.01" length="0.03"/>
