Commit message: Update

File: 4_Wheel/quadwheel/model/connector.xacro (robot description, xacro)
@@ -1,12 +1,14 @@
 <?xml version='1.0'?>
 <robot xmlns:xacro="http://www.ros.org/wiki/xacro">
-<xacro:include filename="$(find gazebo_test)/model/rim.xacro"/>
+<xacro:include filename="$(find quadwheel)/model/rim.xacro"/>
 <xacro:macro name="connector" params="name parent xyz rpy GAZEBO_color">
   <link name="C${name}">
     <inertial>
+      <origin xyz="0 0 -0.0286" rpy="0 0 0" />
       <mass value="0.10"/>
       <inertia ixx="7.6e-5" ixy="0.0" ixz="0.0" iyy="7.6e-5" iyz="0.0" izz="0.000125"/>
     </inertial>
     <visual>
+      <origin xyz="0 0 -0.0286" rpy="0 0 0" />
       <geometry>
         <cylinder radius="0.0318" length="0.0572"/>
@@ -14,14 +16,17 @@
     </visual>
   </link>
-  <joint name="${parent}_C${name}_joint" type="fixed">
+  <joint name="${parent}_C${name}_joint" type="continuous">
     <parent link="${parent}"/>
     <child link="C${name}"/>
     <origin xyz = "${xyz}" rpy = "${rpy}"/>
+    <axis xyz = "0 0 1"/>
   </joint>
   <!--Wheel Rims -->
-  <xacro:rim name="wheel_${name}" parent="C${name}" xyz="0 0 -0.0286" rpy="0 0 0" GAZEBO_color = "Gazebo/Red"/>
-  <gazebo reference="connector_${name}_link">
-    <material value= "${GAZEBO_color}"/>
-  </gazebo>
+  <xacro:rim name="wheel_${name}" parent="C${name}" xyz="0 0 -0.0572" rpy="0 0 0" GAZEBO_color = "${GAZEBO_color}"/>
+<gazebo reference="C${name}">
+  <mu>0.2</mu>
+  <mu2>0.2</mu2>
+  <material value= "${GAZEBO_color}"/>
+</gazebo>
 </xacro:macro>
 </robot>

File: 4_Wheel/quadwheel/model/roller.xacro (robot description, xacro)
@@ -1,11 +1,13 @@
 <?xml version='1.0'?>
 <robot xmlns:xacro="http://www.ros.org/wiki/xacro">
-<xacro:macro name="roller" params="name parent xyz rpy">
+<xacro:macro name="roller" params="name parent xyz rpy GAZEBO_color">
   <link name="roller_${name}_rim_${parent}_link">
     <inertial>
+      <origin xyz="0 -0.0182 0" rpy="0 0 0" />
       <inertia ixx="1e-6" ixy="0.0" ixz="0.0" iyy="1e-6" iyz="0.0" izz="1e-7"/>
       <mass value="0.010"/>
     </inertial>
     <visual>
+      <origin xyz="0 -0.0182 0" rpy="0 0 0" />
       <geometry>
         <cylinder radius="0.01" length="0.03"/>
@@ -13,4 +15,5 @@
     </visual>
     <collision>
+      <origin xyz="0 -0.0182 0" rpy="0 0 0" />
       <geometry>
         <cylinder radius="0.01" length="0.03"/>
@@ -25,4 +28,9 @@
     <limit effort="1000" velocity="31.4"/>
   </joint>
+<gazebo reference="roller_${name}_rim_${parent}_link">
+  <mu>0.2</mu>
+  <mu2>0.2</mu2>
+  <material value= "${GAZEBO_color}"/>
+</gazebo>
 </xacro:macro>
 </robot>

Commit message: controller update

File: 4_Wheel/quadwheel/model/connector.xacro (robot description, xacro)
@@ -21,12 +21,11 @@
     <origin xyz = "${xyz}" rpy = "${rpy}"/>
     <axis xyz = "0 0 1"/>
+    <limit velocity="1.0" effort="30" />
   </joint>
-  <!--Wheel Rims -->
+  <!-- Wheel Rims -->
   <xacro:rim name="wheel_${name}" parent="C${name}" xyz="0 0 -0.0572" rpy="0 0 0" GAZEBO_color = "${GAZEBO_color}"/>
-<gazebo reference="C${name}">
-  <mu>0.2</mu>
-  <mu2>0.2</mu2>
-  <material value= "${GAZEBO_color}"/>
-</gazebo>
+  <gazebo reference="C${name}">
+    <material value= "${GAZEBO_color}"/>
+  </gazebo>
 </xacro:macro>
 </robot>

File: 4_Wheel/quadwheel/model/main.xacro (robot description, xacro)
@@ -2,5 +2,4 @@
 <robot name="4_wheel_omni" xmlns:xacro="http://www.ros.org/wiki/xacro">
   <xacro:include filename="$(find quadwheel)/model/connector.xacro"/>
-  <xacro:include filename="$(find quadwheel)/model/plugins.gazebo"/>
   <!-- World Link -->
   <link name="base_link" />
@@ -26,4 +25,7 @@
     </inertial>
   </link>
+  <gazebo reference="chassis">
+    <material value= "Gazebo/Green"/>
+  </gazebo>
   <!--Wheel Rims -->
   <xacro:connector name="1" parent="chassis" xyz="0.228 0.228 0.01" rpy="1.57 0 -0.7854" GAZEBO_color = "Gazebo/Red"/>
@@ -31,44 +33,5 @@
   <xacro:connector name="3" parent="chassis" xyz="-0.228 -0.228 0.01" rpy="1.57 0 -3.9270" GAZEBO_color = "Gazebo/Green"/>
   <xacro:connector name="4" parent="chassis" xyz="-0.228 0.228 0.01" rpy="1.57 0 -5.4978" GAZEBO_color = "Gazebo/Yellow"/>
-  <!-- Motors -->
-  <transmission name="tran1">
-    <type>transmission_interface/SimpleTransmission</type>
-    <joint name="chassis_C1_joint">
-      <hardwareInterface>hardware_interface/EffortJointInterface</hardwareInterface>
-    </joint>
-    <actuator name="motor1">
-      <hardwareInterface>hardware_interface/EffortJointInterface</hardwareInterface>
-      <mechanicalReduction>1</mechanicalReduction>
-    </actuator>
-  </transmission>
-  <transmission name="tran2">
-    <type>transmission_interface/SimpleTransmission</type>
-    <joint name="chassis_C2_joint">
-      <hardwareInterface>hardware_interface/EffortJointInterface</hardwareInterface>
-    </joint>
-    <actuator name="motor2">
-      <hardwareInterface>hardware_interface/EffortJointInterface</hardwareInterface>
-      <mechanicalReduction>1</mechanicalReduction>
-    </actuator>
-  </transmission>
-  <transmission name="tran3">
-    <type>transmission_interface/SimpleTransmission</type>
-    <joint name="chassis_C3_joint">
-      <hardwareInterface>hardware_interface/EffortJointInterface</hardwareInterface>
-    </joint>
-    <actuator name="motor3">
-      <hardwareInterface>hardware_interface/EffortJointInterface</hardwareInterface>
-      <mechanicalReduction>1</mechanicalReduction>
-    </actuator>
-  </transmission>
-  <transmission name="tran4">
-    <type>transmission_interface/SimpleTransmission</type>
-    <joint name="chassis_C4_joint">
-      <hardwareInterface>hardware_interface/EffortJointInterface</hardwareInterface>
-    </joint>
-    <actuator name="motor4">
-      <hardwareInterface>hardware_interface/EffortJointInterface</hardwareInterface>
-      <mechanicalReduction>1</mechanicalReduction>
-    </actuator>
-  </transmission>
+  <!-- Control -->
+  <xacro:include filename="$(find quadwheel)/model/ros2_control.xacro"/>
 </robot>

File: 4_Wheel/quadwheel/model/rim.xacro (robot description, xacro)
@@ -41,6 +41,4 @@
 <xacro:roller name="18" parent="${name}"  xyz="0.0390 -0.0142 -0.008" rpy="1.57 0 5.9341" GAZEBO_color = "${GAZEBO_color}"/>
 <gazebo reference="rim_${name}_link">
-  <mu>0.2</mu>
-  <mu2>0.2</mu2>
   <material value= "${GAZEBO_color}"/>
 </gazebo>

File: 4_Wheel/quadwheel/model/roller.xacro (robot description, xacro)
@@ -1,5 +1,5 @@
 <?xml version='1.0'?>
 <robot xmlns:xacro="http://www.ros.org/wiki/xacro">
-<xacro:macro name="roller" params="name parent xyz rpy GAZEBO_color">
+  <xacro:macro name="roller" params="name parent xyz rpy GAZEBO_color">
   <link name="roller_${name}_rim_${parent}_link">
     <inertial>
@@ -28,9 +28,9 @@
     <limit effort="1000" velocity="31.4"/>
   </joint>
-<gazebo reference="roller_${name}_rim_${parent}_link">
-  <mu>0.2</mu>
-  <mu2>0.2</mu2>
-  <material value= "${GAZEBO_color}"/>
-</gazebo>
-</xacro:macro>
+  <gazebo reference="roller_${name}_rim_${parent}_link">
+    <mu1 value="0.001"/>
+    <mu2 value="0.002"/>
+    <material value= "Gazebo/Grey"/>
+  </gazebo>
+  </xacro:macro>
 </robot>

File: 4_Wheel/quadwheel/model/ros2_control.xacro (robot description, xacro)
@@ -39,5 +39,5 @@
     </ros2_control>
     <gazebo>
-        <plugin name="gz_ros2_control::GazeboSimROS2ControlPlugin" filename="libgz_ros2_control-system.so">
+        <plugin name="gz_ros2_control::GazeboSimROS2ControlPlugin" filename="gz_ros2_control-system">
             <parameters>$(find quadwheel)/config/my_controllers.yaml</parameters>
         </plugin>
